Commit message: Model with sun finger

File: sun_wsg50_simulation/urdf/gripper_wsg50.urdf.xacro (robot description, xacro)
@@ -8,5 +8,5 @@
   <xacro:arg name="robot_name" default="gripper"/>
   <xacro:arg name="origin_xyz" default="0 0 0.851"/>
-  <xacro:arg name="origin_rpy" default="0 0 0"/>
+  <xacro:arg name="origin_rpy" default="-1.5707 0 0"/>
   <material name="workcell">
     <color rgba="0.8 1.0 0.8 0.2"/>
@@ -16,6 +16,35 @@
   </link>
   <!--iiwa-->
-  <xacro:wsg50 hardware_interface="$(arg hardware_interface)" robot_name="$(arg robot_name)" parent="world">
+  <xacro:wsg50
+    hardware_interface="$(arg hardware_interface)"
+    robot_name="$(arg robot_name)"
+    parent="world"
+    scale="15.0"
+    finger_file="case_v2.stl"
+    fingerpx="-0.065"
+    fingerpy="-0.045"
+    fingerpz="0.06"
+    fingeror="1.5707"
+    fingerop="0.0"
+    fingeroy="1.5707"
+    ee_link_z="0.195"
+    >
     <origin xyz="$(arg origin_xyz)" rpy="$(arg origin_rpy)" />
   </xacro:wsg50>
+  <!--xacro:wsg50
+    hardware_interface="$(arg hardware_interface)"
+    robot_name="$(arg robot_name)"
+    parent="world"
+    scale="15.0"
+    finger_file="WSG-FMF.stl"
+    fingerpx="0.0"
+    fingerpy="0.0"
+    fingerpz="0.0"
+    fingeror="0.0"
+    fingerop="0.0"
+    fingeroy="0.0"
+    ee_link_z="0.195"
+    >
+    <origin xyz="$(arg origin_xyz)" rpy="$(arg origin_rpy)" />
+  </xacro:wsg50-->
 </robot>

File: sun_wsg50_simulation/urdf/gripper_wsg50.xacro (robot description, xacro)
@@ -1,5 +1,5 @@
 <?xml version="1.0"?>
 <robot xmlns:xacro="http://www.ros.org/wiki/xacro">
-  <xacro:macro name="wsg50" params="parent hardware_interface robot_name *origin">
+  <xacro:macro name="wsg50" params="parent hardware_interface robot_name *origin scale finger_file fingerpx fingerpy fingerpz fingeror fingerop fingeroy ee_link_z">
     <!--joint between {parent} and gripper_roll_link-->
     <joint name="${parent}_${robot_name}_joint" type="fixed">
@@ -18,5 +18,5 @@
           <origin xyz="0.0 0 0" rpy="0 0 0" />
           <geometry>
-             <mesh filename="package://sun_wsg50_simulation/meshes/WSG50_110.stl" scale="1 1 1"/>
+             <mesh filename="package://sun_wsg50_simulation/meshes/WSG50_110.stl" scale="${scale*1} ${scale*1} ${scale*1}"/>
           </geometry>
           <material name="grey">
@@ -27,5 +27,5 @@
           <origin xyz="0.0 0 0" rpy="0 0 0" />
           <geometry>
-             <mesh filename="package://sun_wsg50_simulation/meshes/WSG50_110.stl" scale="1 1 1"/>
+             <mesh filename="package://sun_wsg50_simulation/meshes/WSG50_110.stl" scale="${scale*1} ${scale*1} ${scale*1}"/>
          </geometry>
      </collision>
@@ -40,5 +40,5 @@
           <origin xyz="0.0 0 0.0" rpy="0 0 0" />
       <geometry>
-             <mesh filename="package://sun_wsg50_simulation/meshes/GUIDE_WSG50_110.stl" scale="0.001 0.001 0.001"/>
+             <mesh filename="package://sun_wsg50_simulation/meshes/GUIDE_WSG50_110.stl" scale="${scale*0.001} ${scale*0.001} ${scale*0.001}"/>
       </geometry>
       <material name="black"/>
@@ -47,5 +47,5 @@
           <origin xyz="0 0 0" rpy="0 0 0" />
       <geometry>
-             <mesh filename="package://sun_wsg50_simulation/meshes/GUIDE_WSG50_110.stl" scale="0.001 0.001 0.001"/>
+             <mesh filename="package://sun_wsg50_simulation/meshes/GUIDE_WSG50_110.stl" scale="${scale*0.001} ${scale*0.001} ${scale*0.001}"/>
       </geometry>
     </collision>
@@ -63,9 +63,9 @@
     <origin xyz="0 0 0"/>
     <axis xyz="1 0 0"/>
-     <limit lower="-0.055" upper="-0.0027" effort="1.0" velocity="1.0"/>
+     <limit lower="${-0.055*scale}" upper="${-0.0027*scale}" effort="1.0" velocity="1.0"/>
     <dynamics damping="50" friction="1"/>
 </joint>
   <joint name="guide_joint_finger_left" type="fixed">
-     <origin xyz="0 0 0.023" rpy="0 0 0" />
+     <origin xyz="0 0 ${0.023*scale}" rpy="0 0 0" />
      <parent link="finger_link1"/>
      <child link="finger_left" />
@@ -76,16 +76,15 @@
   <link name="finger_left">
       <visual>
-          <origin xyz="0.0 0 0.0" rpy="0 0 0" />
+          <origin xyz="${fingerpx*scale} ${fingerpy*scale} ${fingerpz*scale}" rpy="${fingeror} ${fingerop} ${fingeroy}" />
           <geometry>
-             <mesh filename="package://sun_wsg50_simulation/meshes/WSG-FMF.stl" scale="0.001 0.001 0.001"/>
+             <mesh filename="package://sun_wsg50_simulation/meshes/${finger_file}" scale="${scale*0.001} ${scale*0.001} ${scale*0.001}"/>
           </geometry>
-          <material name="black">
-		<color rgba="0 0 0 0"/>
+          <material name="White">
       	  </material>
       </visual>
       <collision>
-          <origin xyz="0 0 0" rpy="0 0 0" />
+          <origin xyz="${fingerpx*scale} ${fingerpy*scale} ${fingerpz*scale}" rpy="${fingeror} ${fingerop} ${fingeroy}" />
           <geometry>
-             <mesh filename="package://sun_wsg50_simulation/meshes/WSG-FMF.stl" scale="0.001 0.001 0.001"/>
+             <mesh filename="package://sun_wsg50_simulation/meshes/${finger_file}" scale="${scale*0.001} ${scale*0.001} ${scale*0.001}"/>
          </geometry>
      </collision>
@@ -99,5 +98,5 @@
       <origin rpy="0 0 0" xyz="0 0 0.0"/>
       <geometry>
-             <mesh filename="package://sun_wsg50_simulation/meshes/GUIDE_WSG50_110.stl" scale="0.001 0.001 0.001"/>
+             <mesh filename="package://sun_wsg50_simulation/meshes/GUIDE_WSG50_110.stl" scale="${scale*0.001} ${scale*0.001} ${scale*0.001}"/>
       </geometry>
       <material name="black"/>
@@ -106,5 +105,5 @@
       <origin rpy="0 0 0" xyz="0 0 0.0"/>
       <geometry>
-             <mesh filename="package://sun_wsg50_simulation/meshes/GUIDE_WSG50_110.stl" scale="0.001 0.001 0.001"/>
+             <mesh filename="package://sun_wsg50_simulation/meshes/GUIDE_WSG50_110.stl" scale="${scale*0.001} ${scale*0.001} ${scale*0.001}"/>
       </geometry>
       <material name="orange"/>
@@ -116,5 +115,5 @@
   </link>
   <joint name="finger_joint2" type="prismatic">
-     <limit lower="0.0027" upper="0.055" effort="1.0" velocity="1.0"/>
+     <limit lower="${0.0027*scale}" upper="${0.055*scale}" effort="1.0" velocity="1.0"/>
      <origin xyz="0 0 0" rpy="0 0 3.14159" />
      <parent link="gripper_roll_link"/>
@@ -125,5 +124,5 @@
   </joint>
   <joint name="guide_joint_finger_right" type="fixed">
-     <origin xyz="0 0 0.023" rpy="0 0 0" />
+     <origin xyz="0 0 ${0.023*scale}" rpy="0 0 0" />
      <parent link="finger_link2"/>
      <child link="finger_right" />
@@ -134,16 +133,15 @@
   <link name="finger_right">
       <visual>
-          <origin xyz="0.0 0 0" rpy="0 0 0" />
+          <origin xyz="${fingerpx*scale} ${fingerpy*scale} ${fingerpz*scale}" rpy="${fingeror} ${fingerop} ${fingeroy}" />
           <geometry>
-             <mesh filename="package://sun_wsg50_simulation/meshes/WSG-FMF.stl" scale="0.001 0.001 0.001"/>
+             <mesh filename="package://sun_wsg50_simulation/meshes/${finger_file}" scale="${scale*0.001} ${scale*0.001} ${scale*0.001}"/>
           </geometry>
-          <material name="black">
-		<color rgba="0 0 0 0"/>
+          <material name="White">
       	  </material>
       </visual>
       <collision>
-          <origin xyz="0 0 0" rpy="0 0 0" />
+          <origin xyz="${fingerpx*scale} ${fingerpy*scale} ${fingerpz*scale}" rpy="${fingeror} ${fingerop} ${fingeroy}" />
           <geometry>
-             <mesh filename="package://sun_wsg50_simulation/meshes/WSG-FMF.stl" scale="0.001 0.001 0.001"/>
+             <mesh filename="package://sun_wsg50_simulation/meshes/${finger_file}" scale="${scale*0.001} ${scale*0.001} ${scale*0.001}"/>
          </geometry>
      </collision>
@@ -154,5 +152,5 @@
       <parent link="gripper_roll_link"/>
       <child link="${robot_name}_link_ee"/>
-      <origin rpy="0 -1.57 0" xyz="0 0 0.22"/>
+      <origin rpy="0 -1.57 0" xyz="0 0 ${ee_link_z*scale}"/>
     </joint>
   </xacro:macro>
