Commit message: add arg to mimic joint

File: sun_wsg50_simulation/urdf/wsg50.urdf.xacro (robot description, xacro)
@@ -1,7 +1,11 @@
 <?xml version="1.0"?>
 <robot name="wsg50" xmlns:xacro="http://www.ros.org/wiki/xacro">
+  <xacro:arg name="scale" default="1.0"/>
+  <xacro:arg name="mimic_joints" default="true"/>
   <!-- Import finger macro -->
   <xacro:include filename="$(find sun_wsg50_simulation)/urdf/wsg50.xacro" />
-  <xacro:wsg50>
-  </xacro:wsg50>
+  <xacro:wsg50
+    scale="$(arg scale)"
+    mimic_joints="$(arg mimic_joints)"
+  />
 </robot>

File: sun_wsg50_simulation/urdf/wsg50.xacro (robot description, xacro)
@@ -11,4 +11,5 @@
         finger_right_name:=finger_right
         scale:=1.0
+        mimic_joints:=true
         "
 >
@@ -42,4 +43,5 @@
     </collision>
 </link>
+<xacro:if value="${mimic_joints}">
 <xacro:wsg50_real_single_joint
     name_prefix=""
@@ -48,10 +50,15 @@
     scale="${scale}"
 />
+<xacro:property name="joint_to_mimic" value="${name_prefix}real_single_joint"/>
+</xacro:if>
+<xacro:unless value="${mimic_joints}">
+<xacro:property name="joint_to_mimic" value="''"/>
+</xacro:unless>
 <xacro:wsg50_finger_flange_with_joint
     name="${finger_left_name}"
     parent_link_name="${name_prefix}${roll_link_name}"
     scale="${scale}"
-    limit_sign="-1.0"
-    joint_to_mimic="${name_prefix}real_single_joint"
+    limit_sign="1.0"
+    joint_to_mimic="${joint_to_mimic}"
     mimic_multipler="0.5"
 >
@@ -64,5 +71,5 @@
     scale="${scale}"
     limit_sign="1.0"
-    joint_to_mimic="${name_prefix}real_single_joint"
+    joint_to_mimic="${joint_to_mimic}"
     mimic_multipler="0.5"
 >
@@ -70,32 +77,4 @@
 <axis xyz="-1 0 0"/>
 </xacro:wsg50_finger_flange_with_joint>
-<!--
-<xacro:property name="finger_cad_file" value="package://sun_tactile_simulation/meshes/sun_finger_v3.stl"/>
-<xacro:property name="cad_scale" value="0.001"/>
-<xacro:property name="local_scale" value="${cad_scale*scale}"/>
-<xacro:property name="finger_mesh">
-  <mesh
-    filename="${finger_cad_file}"
-    scale="${local_scale} ${local_scale} ${local_scale}"
-  />
-</xacro:property>
-<xacro:property name="mesh_origin">
-  <origin xyz="${-56.9550247192*local_scale} ${-45.514275551*local_scale} ${0.00445556640625*local_scale}" rpy="${pi/2.0} ${0.0} ${pi/2}" />
-</xacro:property>
-<link name="${link_name}">
-    <visual>
-        <xacro:insert_block name="mesh_origin" />
-        <geometry>
-            <xacro:insert_block name="finger_mesh" />
-        </geometry>
-    </visual>
-    <collision>
-        <xacro:insert_block name="mesh_origin" />
-        <geometry>
-            <xacro:insert_block name="finger_mesh" />
-         </geometry>
-     </collision>
-</link>
--->
 </xacro:macro>
 </robot>
