Commit message: Add color

File: sun_wsg50_simulation/urdf/finger_flange.xacro (robot description, xacro)
@@ -29,4 +29,7 @@
             <xacro:insert_block name="wsg50_finger_flange_mesh" />
         </geometry>
+        <material name="black">
+            <color rgba="0 0 0 1"/>
+        </material>
     </visual>
     <collision>

File: sun_wsg50_simulation/urdf/wsg50.xacro (robot description, xacro)
@@ -31,4 +31,7 @@
             <xacro:insert_block name="wsg50_110_mesh" />
         </geometry>
+        <material name="gray">
+            <color rgba="0.5 0.5 0.5 1"/>
+        </material>
     </visual>
     <collision>

Commit message: use convention for naming

File: sun_wsg50_simulation/urdf/finger_flange.xacro (robot description, xacro)
@@ -3,89 +3,136 @@
 <xacro:property name="finger_joint_limit_lower" value="0.0"/>
 <xacro:property name="finger_joint_limit_upper" value="0.110"/>
-<!-- macro for finger flange -->
+<!--
+    MACRO to generate finger flange (sensor port)
+    base_link = name of the link (default base_link)
+    scale = unit scale, 1.0 = [m] (default 1.0)
+    prefix = name to use prefix (default '')
+    the finger flange link will be ${prefix}${base_link}
+-->
 <xacro:macro
     name="wsg50_finger_flange"
     params="
-        link_name:=finger_link
+        base_link:=base_link
         scale:=1.0
+        prefix:=''
         "
 >
-<xacro:property name="wsg50_finger_flange_cad_file" value="package://sun_wsg50_simulation/meshes/GUIDE_WSG50_110.stl"/>
-<xacro:property name="cad_scale" value="0.001"/>
-<xacro:property name="local_scale" value="${cad_scale*scale}"/>
-<xacro:property name="wsg50_finger_flange_mesh">
-    <mesh
-        filename="${wsg50_finger_flange_cad_file}"
-        scale="${local_scale} ${local_scale} ${local_scale}"
-    />
-</xacro:property>
-<xacro:property name="wsg50_finger_flange_mesh_origin">
-    <origin xyz="${0.0*local_scale} ${0.0*local_scale} ${0.0*local_scale}" rpy="${0.0} ${0.0} ${0.0}" />
-</xacro:property>
-<link name="${link_name}">
-    <visual>
-        <xacro:insert_block name="wsg50_finger_flange_mesh_origin" />
-        <geometry>
-            <xacro:insert_block name="wsg50_finger_flange_mesh" />
-        </geometry>
-        <material name="black">
-            <color rgba="0 0 0 1"/>
-        </material>
-    </visual>
-    <collision>
-        <xacro:insert_block name="wsg50_finger_flange_mesh_origin" />
-        <geometry>
-            <xacro:insert_block name="wsg50_finger_flange_mesh" />
-        </geometry>
-    </collision>
-</link>
-</xacro:macro>
-<!-- MACRO THAT IMPLEMENTS THE REAL SINGLE JOINT OF THE GRIPPER -->
-<xacro:macro
-    name="wsg50_real_single_joint"
-    params="
-        name_prefix:=''
-        name:=real_single_joint
-        parent_link_name:=gripper_roll_link
-        scale:=1.0
-        "
->
-<joint name="${name_prefix}${name}" type="prismatic">
-    <parent link="${parent_link_name}"/>
-    <child link="${name_prefix}${name}_fake_link"/>
-    <limit lower="${finger_joint_limit_lower*scale}" upper="${finger_joint_limit_upper*scale}" effort="1.0" velocity="1.0"/>
-</joint>
-<link name="${name_prefix}${name}_fake_link">
-</link>
-</xacro:macro>
-<!-- macro for finger flange with joint -->
+    <!-- cad_scale to convert from cad to [m] -->
+    <xacro:property name="cad_scale" value="0.001"/>
+    <!-- local_scale cad to input scale -->
+    <xacro:property name="local_scale" value="${cad_scale*scale}"/>
+    <!-- origin of mesh wrt link frame -->
+    <xacro:property name="wsg50_finger_flange_mesh_origin">
+        <origin
+            xyz="${0.0*local_scale} ${0.0*local_scale} ${0.0*local_scale}"
+            rpy="${0.0} ${0.0} ${0.0}"
+        />
+    </xacro:property>
+    <!-- finger flange link -->
+    <link name="${prefix}${base_link}">
+        <visual>
+            <xacro:insert_block name="wsg50_finger_flange_mesh_origin" />
+            <geometry>
+                <mesh
+                    filename="package://sun_wsg50_simulation/meshes/visual/GUIDE_WSG50_110.stl"
+                    scale="${local_scale} ${local_scale} ${local_scale}"
+                />
+            </geometry>
+            <material name="black">
+                <color rgba="0 0 0 1"/>
+            </material>
+        </visual>
+        <collision>
+            <xacro:insert_block name="wsg50_finger_flange_mesh_origin" />
+            <geometry>
+                <mesh
+                    filename="package://sun_wsg50_simulation/meshes/collision/GUIDE_WSG50_110.stl"
+                    scale="${local_scale} ${local_scale} ${local_scale}"
+                />
+            </geometry>
+        </collision>
+    </link>
+</xacro:macro> <!-- end macro finger flange link -->
+<!--
+    MACRO to generate finger flange (sensor port) with prismatic joint
+    prefix = name to use prefix (default '')
+    scale = unit scale, 1.0 = [m] (default 1.0)
+    joint_name = joint name for the prismatic joint (default finger_flange_joint)
+    parent_link = parent link to attach (default wsg50/base_link)
+    finger_flange_link = link name to use for the finger flange (sensor port) (default finger_flange_link)
+    joint_to_mimic = joint to mimic, if '' no mimic (default '')
+    mimic_multipler = multipler to use in mimic (default 0.5)
+    limit_sign = joint limit sign (you should not use di arg) (default 1.0)
+    *link_origin = origin tag for the prismatic joint
+    the finger flange link will be ${prefix}${finger_flange_link}
+    the prismatic joint will be ${prefix}${joint_name}
+-->
 <xacro:macro
     name="wsg50_finger_flange_with_joint"
     params="
-        name:=finger
-        parent_link_name:=gripper_roll_link
+        prefix:=''
         scale:=1.0
-        limit_sign:=-1.0
+        joint_name:=finger_flange_joint
+        parent_link:=wsg50/base_link
+        finger_flange_link:=finger_flange_link
         joint_to_mimic:=''
         mimic_multipler:=0.5
+        limit_sign:=1.0
         *link_origin
-        *link_axis
         "
 >
-<joint name="${name}_joint" type="prismatic">
-    <parent link="${parent_link_name}"/>
-    <child link="${name}_link"/>
-    <xacro:insert_block name="link_origin" />
-    <xacro:insert_block name="link_axis" />
-    <!--limit lower="${limit_sign*(1+0*0.055)*scale}" upper="${limit_sign*(0+0*0.0027)*scale}" effort="1.0" velocity="1.0"/-->
-    <limit lower="${limit_sign*(finger_joint_limit_lower/2)*scale}" upper="${limit_sign*(finger_joint_limit_upper/2)*scale}" effort="1.0" velocity="1.0"/>
-    <xacro:unless value="${joint_to_mimic==''}">
-        <mimic joint="${joint_to_mimic}" multiplier="${mimic_multipler}" offset="0" />
-    </xacro:unless>
-</joint>
-<xacro:wsg50_finger_flange
-    link_name="${name}_link"
-    scale="${scale}"
-/>
-</xacro:macro>
+    <!-- Prismatic joint -->
+    <joint name="${prefix}${joint_name}" type="prismatic">
+        <parent link="${parent_link}"/>
+        <child link="${prefix}${finger_flange_link}"/>
+        <xacro:insert_block name="link_origin" />
+        <axis xyz="-1 0 0"/>
+        <limit
+            lower="${limit_sign*(finger_joint_limit_lower/2)*scale}"
+            upper="${limit_sign*(finger_joint_limit_upper/2)*scale}"
+            effort="1.0" velocity="1.0"
+        />
+        <xacro:unless value="${joint_to_mimic==''}">
+            <mimic joint="${joint_to_mimic}" multiplier="${mimic_multipler}" offset="0" />
+        </xacro:unless>
+    </joint>
+    <!-- finger flange link -->
+    <xacro:wsg50_finger_flange
+        base_link="${finger_flange_link}"
+        scale="${scale}"
+        prefix="${prefix}"
+    />
+</xacro:macro> <!-- end macro finger flange + prismatic joint -->
+<!-- MACRO THAT IMPLEMENTS THE REAL SINGLE JOINT OF THE GRIPPER -->
+<!--
+    MACRO to generate a fake joint/link that represents the real 1DOF joint of wsg50
+    prefix = name to use prefix (default '')
+    scale = unit scale, 1.0 = [m] (default 1.0)
+    joint_name = joint name for the prismatic joint (default 1dof_joint)
+    parent_link = parent link to attach (default wsg50/base_link)
+    the prismatic joint will be ${prefix}${joint_name}
+    this fake joint is usefull with the arg joint_to_mimic of wsg50_finger_flange_with_joint
+-->
+<xacro:macro
+    name="wsg50_1dof_joint"
+    params="
+        prefix:=''
+        scale:=1.0
+        joint_name:=1dof_joint
+        parent_link:=wsg50/base_link
+        "
+>
+    <!-- Prismatic joint -->
+    <joint name="${prefix}${joint_name}" type="prismatic">
+        <parent link="${parent_link}"/>
+        <child link="${prefix}${joint_name}_fake_link"/>
+        <limit
+            lower="${finger_joint_limit_lower*scale}"
+            upper="${finger_joint_limit_upper*scale}"
+            effort="1.0" velocity="1.0"
+        />
+    </joint>
+    <!-- fake link -->
+    <link name="${prefix}${joint_name}_fake_link"/>
+</xacro:macro> <!-- end macro 1dof_joint -->
 </robot>

File: sun_wsg50_simulation/urdf/wsg50.urdf.xacro (robot description, xacro)
@@ -1,11 +1,15 @@
 <?xml version="1.0"?>
 <robot name="wsg50" xmlns:xacro="http://www.ros.org/wiki/xacro">
-  <xacro:arg name="scale" default="1.0"/>
-  <xacro:arg name="mimic_joints" default="true"/>
-  <!-- Import finger macro -->
+  <!-- Import wsg50 macro -->
   <xacro:include filename="$(find sun_wsg50_simulation)/urdf/wsg50.xacro" />
   <xacro:wsg50
-    scale="$(arg scale)"
-    mimic_joints="$(arg mimic_joints)"
+    prefix="''"
+    scale="1.0"
+    base_link="base_link"
+    mimic_joints="true"
+    prefix_finger_left="left/"
+    finger_flange_left_link="finger_flange_link"
+    prefix_finger_right="right/"
+    finger_flange_right_link="finger_flange_link"
   />
 </robot>

File: sun_wsg50_simulation/urdf/wsg50.xacro (robot description, xacro)
@@ -1,80 +1,114 @@
 <?xml version="1.0"?>
 <robot xmlns:xacro="http://www.ros.org/wiki/xacro">
-<!-- Import finger flange macro -->
+<!-- Import finger flange macros -->
 <xacro:include filename="$(find sun_wsg50_simulation)/urdf/finger_flange.xacro" />
+<!--
+    MACRO to generate wsg50 without fingers
+    prefix = name to use as prefix (default '')
+    scale = unit scale, 1.0 = [m] (default 1.0)
+    base_link = base link of the gripper (default base_link)
+    mimic_joints = if true, create a fake joint for the real 1dof joint of the gripper and ad mimic tag to the 2 prismatic joints (default true)
+    prefix_finger_left = prefix to use fot the left finger (default left/)
+    prefix_finger_left = prefix to use fot the left finger (default left/)
+    finger_flange_left_link = link name for the left finger flange (default finger_flange_link)
+    prefix_finger_right = prefix to use fot the right finger (default right/)
+    finger_flange_right_link = link name for the right finger flange (default finger_flange_link)
+    the gripper base link will be ${prefix}${base_link}
+    the two prismatic joints : ${prefix}${prefix_finger_left}finger_flange_joint and ${prefix}${prefix_finger_right}finger_flange_joint
+    if mimic_joints=true the fake 1dof joint will be ${prefix}1dof_joint
+-->
 <xacro:macro
     name="wsg50"
     params="
-        name_prefix:=''
-        roll_link_name:=gripper_roll_link
-        finger_left_name:=finger_left
-        finger_right_name:=finger_right
+        prefix:=''
         scale:=1.0
+        base_link:=base_link
         mimic_joints:=true
+        prefix_finger_left:=left/
+        finger_flange_left_link:=finger_flange_link
+        prefix_finger_right:=right/
+        finger_flange_right_link:=finger_flange_link
         "
 >
-<xacro:property name="wsg50_110_cad_file" value="package://sun_wsg50_simulation/meshes/WSG50_110.stl"/>
-<xacro:property name="cad_scale" value="1.0"/>
-<xacro:property name="local_scale" value="${cad_scale*scale}"/>
-<xacro:property name="wsg50_110_mesh">
-  <mesh
-    filename="${wsg50_110_cad_file}"
-    scale="${local_scale} ${local_scale} ${local_scale}"
-  />
-</xacro:property>
-<xacro:property name="wsg50_110_mesh_origin">
-  <origin xyz="${0.0*local_scale} ${0.0*local_scale} ${0.0*local_scale}" rpy="${0.0} ${0.0} ${0.0}" />
-</xacro:property>
-<link name="${name_prefix}${roll_link_name}">
-    <visual>
-        <xacro:insert_block name="wsg50_110_mesh_origin" />
-        <geometry>
-            <xacro:insert_block name="wsg50_110_mesh" />
-        </geometry>
-        <material name="gray">
-            <color rgba="0.5 0.5 0.5 1"/>
-        </material>
-    </visual>
-    <collision>
-        <xacro:insert_block name="wsg50_110_mesh_origin" />
-        <geometry>
-            <xacro:insert_block name="wsg50_110_mesh" />
-        </geometry>
-    </collision>
-</link>
-<xacro:if value="${mimic_joints}">
-<xacro:wsg50_real_single_joint
-    name_prefix=""
-    name="${name_prefix}gripper_joint"
-    parent_link_name="${name_prefix}${roll_link_name}"
-    scale="${scale}"
-/>
-<xacro:property name="joint_to_mimic" value="${name_prefix}gripper_joint"/>
-</xacro:if>
-<xacro:unless value="${mimic_joints}">
-<xacro:property name="joint_to_mimic" value="''"/>
-</xacro:unless>
-<xacro:wsg50_finger_flange_with_joint
-    name="${finger_left_name}"
-    parent_link_name="${name_prefix}${roll_link_name}"
-    scale="${scale}"
-    limit_sign="1.0"
-    joint_to_mimic="${joint_to_mimic}"
-    mimic_multipler="0.5"
->
-<origin xyz="0 0 0" rpy="0 0 0.0"/>
-<axis xyz="-1 0 0"/>
-</xacro:wsg50_finger_flange_with_joint>
-<xacro:wsg50_finger_flange_with_joint
-    name="${finger_right_name}"
-    parent_link_name="${name_prefix}${roll_link_name}"
-    scale="${scale}"
-    limit_sign="1.0"
-    joint_to_mimic="${joint_to_mimic}"
-    mimic_multipler="0.5"
->
-<origin xyz="0 0 0" rpy="0 0 ${pi}"/>
-<axis xyz="-1 0 0"/>
-</xacro:wsg50_finger_flange_with_joint>
-</xacro:macro>
+    <!-- cad_scale to convert from cad to [m] -->
+    <xacro:property name="cad_scale" value="1.0"/>
+    <!-- local_scale cad to input scale -->
+    <xacro:property name="local_scale" value="${cad_scale*scale}"/>
+    <!-- origin of mesh wrt link frame -->
+    <xacro:property name="wsg50_110_mesh_origin">
+        <origin
+            xyz="${0.0*local_scale} ${0.0*local_scale} ${0.0*local_scale}"
+            rpy="${0.0} ${0.0} ${0.0}"
+        />
+    </xacro:property>
+    <!-- WSG50 base_link of the gripper -->
+    <link name="${prefix}${base_link}">
+        <visual>
+            <xacro:insert_block name="wsg50_110_mesh_origin" />
+            <geometry>
+                <mesh
+                    filename="package://sun_wsg50_simulation/meshes/visual/WSG50_110.stl"
+                    scale="${local_scale} ${local_scale} ${local_scale}"
+                />
+            </geometry>
+            <material name="gray">
+                <color rgba="0.5 0.5 0.5 1"/>
+            </material>
+        </visual>
+        <collision>
+            <xacro:insert_block name="wsg50_110_mesh_origin" />
+            <geometry>
+                <mesh
+                    filename="package://sun_wsg50_simulation/meshes/collision/WSG50_110.stl"
+                    scale="${local_scale} ${local_scale} ${local_scale}"
+                />
+            </geometry>
+        </collision>
+    </link> <!-- end wsg50 base link -->
+    <!-- check if I must mimic the joints -->
+    <xacro:if value="${mimic_joints}">
+        <!-- mimic the joints -> create a fake 1dof joint -->
+        <xacro:wsg50_1dof_joint
+            prefix="${prefix}"
+            scale="${scale}"
+            joint_name="1dof_joint"
+            parent_link="${prefix}${base_link}"
+        />
+        <!-- prepare the property joint_to_mimic for finger flange macro -->
+        <xacro:property name="joint_to_mimic" value="${prefix}1dof_joint"/>
+    </xacro:if>
+    <xacro:unless value="${mimic_joints}">
+        <xacro:property name="joint_to_mimic" value="''"/>
+    </xacro:unless>
+    <!-- finger flange + link (left) -->
+        <!--
+            joint_name=default
+            limit_sign=default
+            mimic_multipler=default
+        -->
+    <xacro:wsg50_finger_flange_with_joint
+        prefix="${prefix}${prefix_finger_left}"
+        scale="${scale}"
+        parent_link="${prefix}${base_link}"
+        joint_to_mimic="${joint_to_mimic}"
+        finger_flange_link="${finger_flange_left_link}"
+    >
+        <origin xyz="0 0 0" rpy="0 0 0"/>
+    </xacro:wsg50_finger_flange_with_joint>
+    <!-- finger flange + link (right) -->
+        <!--
+            joint_name=default
+            limit_sign=default
+            mimic_multipler=default
+        -->
+    <xacro:wsg50_finger_flange_with_joint
+        prefix="${prefix}${prefix_finger_right}"
+        scale="${scale}"
+        parent_link="${prefix}${base_link}"
+        joint_to_mimic="${joint_to_mimic}"
+        finger_flange_link="${finger_flange_right_link}"
+    >
+        <origin xyz="0 0 0" rpy="0 0 ${pi}"/>
+    </xacro:wsg50_finger_flange_with_joint>
+</xacro:macro> <!-- end macro wsg50 -->
 </robot>

Commit message: change default joint name, add grasp force visualizer

File: sun_wsg50_simulation/urdf/finger_flange.xacro (robot description, xacro)
@@ -109,5 +109,5 @@
     prefix = name to use prefix (default '')
     scale = unit scale, 1.0 = [m] (default 1.0)
-    joint_name = joint name for the prismatic joint (default 1dof_joint)
+    joint_name = joint name for the prismatic joint (default gripper_joint)
     parent_link = parent link to attach (default wsg50/base_link)
     the prismatic joint will be ${prefix}${joint_name}
@@ -119,5 +119,5 @@
         prefix:=''
         scale:=1.0
-        joint_name:=1dof_joint
+        joint_name:=gripper_joint
         parent_link:=wsg50/base_link
         "

File: sun_wsg50_simulation/urdf/wsg50.xacro (robot description, xacro)
@@ -16,5 +16,5 @@
     the gripper base link will be ${prefix}${base_link}
     the two prismatic joints : ${prefix}${prefix_finger_left}finger_flange_joint and ${prefix}${prefix_finger_right}finger_flange_joint
-    if mimic_joints=true the fake 1dof joint will be ${prefix}1dof_joint
+    if mimic_joints=true the fake 1dof joint will be ${prefix}gripper_joint
 -->
 <xacro:macro
@@ -72,9 +72,9 @@
             prefix="${prefix}"
             scale="${scale}"
-            joint_name="1dof_joint"
+            joint_name="gripper_joint"
             parent_link="${prefix}${base_link}"
         />
         <!-- prepare the property joint_to_mimic for finger flange macro -->
-        <xacro:property name="joint_to_mimic" value="${prefix}1dof_joint"/>
+        <xacro:property name="joint_to_mimic" value="${prefix}gripper_joint"/>
     </xacro:if>
     <xacro:unless value="${mimic_joints}">
