Commit message: change default mimic joint to gripper_joint

File: sun_wsg50_simulation/urdf/wsg50.xacro (robot description, xacro)
@@ -46,9 +46,9 @@
 <xacro:wsg50_real_single_joint
     name_prefix=""
-    name="${name_prefix}real_single_joint"
+    name="${name_prefix}gripper_joint"
     parent_link_name="${name_prefix}${roll_link_name}"
     scale="${scale}"
 />
-<xacro:property name="joint_to_mimic" value="${name_prefix}real_single_joint"/>
+<xacro:property name="joint_to_mimic" value="${name_prefix}gripper_joint"/>
 </xacro:if>
 <xacro:unless value="${mimic_joints}">

Commit message: fix collision meshes

File: sun_wsg50_simulation/urdf/wsg50.xacro (robot description, xacro)
@@ -35,4 +35,5 @@
     <!-- local_scale cad to input scale -->
     <xacro:property name="local_scale" value="${cad_scale*scale}"/>
+    <xacro:property name="local_scale_collision" value="${0.001*scale}"/>
     <!-- origin of mesh wrt link frame -->
     <xacro:property name="wsg50_110_mesh_origin">
@@ -61,5 +62,5 @@
                 <mesh
                     filename="package://sun_wsg50_simulation/meshes/collision/WSG50_110.stl"
-                    scale="${local_scale} ${local_scale} ${local_scale}"
+                    scale="${local_scale_collision} ${local_scale_collision} ${local_scale_collision}"
                 />
             </geometry>
